File: eagle/line-sensor-basic/ukmarsbot-line-sensor-basic.sch (EAGLE design)
At the start: 25 parts, among them Q1 PN2222A*, T1 BPW96B, T2 BPW96B, T3 BPW96B, T4 BPW96B

Commit message: Update Line Sensor Basic and library with larger pads/holes for parts
Parts:
- Q1: value PN2222A* -> BC337*
Other:
- note added: "REV B - Nov 2020 - enlarge pads/holes"
Changed lines of the file:
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@@
 <part name="R2" library="ukmarsbot" deviceset="R-EU_" device="0207/7" value="10K"/>
 <part name="C1" library="ukmarsbot" deviceset="CPOL-EU" device="E2.5-7" value="100uF"/>
-<part name="Q1" library="ukmarsbot" deviceset="TRANS_NPN" device="" value="PN2222A*"/>
+<part name="Q1" library="ukmarsbot" deviceset="TRANS_NPN" device="" value="BC337*"/>
 <part name="J2" library="ukmarsbot" deviceset="CONN_03" device=""/>
 <part name="SUPPLY2" library="ukmarsbot" deviceset="5V" device=""/>
@@
 Possible alternatives include BC337-16, ZTX451, ZTX651, ZTX689B.
 </text>
+<text x="114.3" y="-25.4" size="1.778" layer="94">REV B - Nov 2020 - enlarge pads/holes</text>
 </plain>
 <instances>

Commit message: Removed references to depracated SFH4550
Parts:
- LED1, LED2, LED3: value SFH4550 -> Emitter
Other:
- note added: "REV C - Dec 2020 - enlarge pads/holes & Generic emitters"
- note removed: "REV B - Nov 2020 - enlarge pads/holes"
Changed lines of the file:
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@@
 <?xml version="1.0" encoding="utf-8"?>
 <!DOCTYPE eagle SYSTEM "eagle.dtd">
-<eagle version="7.6.0">
+<eagle version="7.5.0">
 <drawing>
 <settings>
@@
 </classes>
 <parts>
-<part name="LED1" library="ukmarsbot" deviceset="LED" device="5MM" value="SFH4550"/>
-<part name="LED2" library="ukmarsbot" deviceset="LED" device="5MM" value="SFH4550"/>
-<part name="LED3" library="ukmarsbot" deviceset="LED" device="5MM" value="SFH4550"/>
+<part name="LED1" library="ukmarsbot" deviceset="LED" device="5MM" value="Emitter"/>
+<part name="LED2" library="ukmarsbot" deviceset="LED" device="5MM" value="Emitter"/>
+<part name="LED3" library="ukmarsbot" deviceset="LED" device="5MM" value="Emitter"/>
 <part name="R3" library="ukmarsbot" deviceset="R-EU_" device="0207/7" value="68R"/>
 <part name="R4" library="ukmarsbot" deviceset="R-EU_" device="0207/7" value="68R"/>
@@
 Possible alternatives include BC337-16, ZTX451, ZTX651, ZTX689B.
 </text>
-<text x="114.3" y="-25.4" size="1.778" layer="94">REV B - Nov 2020 - enlarge pads/holes</text>
+<text x="114.3" y="-25.4" size="1.778" layer="94">REV C - Dec 2020 - enlarge pads/holes &amp; Generic emitters</text>
 </plain>
 <instances>
