File: kicad/line-sensor-mini/line-sensor-mini.kicad_sch (KiCad schematic)
At the start: 25 parts, among them J1 SENSORS, Q1 BC337, Q2 Q_Photo_NPN, Q3 Q_Photo_NPN, Q4 Q_Photo_NPN, Q5 Q_Photo_NPN

Commit message: rename to line-sensor-mini
Parts:
- added R12: 33R, Resistor_THT:R_Axial_DIN0207_L6.3mm_D2.5mm_P7.62mm_Horizontal, symbol Device:R
Connections:
- net +5V: now also R12.2; no longer C1.1, R1.2, R2.1, R3.2
- new net 5V_EMITTERS: C1.1, R1.2, R12.1, R2.1, R3.2
Changed lines of the file:
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@@
   (junction (at 139.7 115.57) (diameter 0) (color 0 0 0 0)
   )
+  (junction (at 107.95 25.4) (diameter 0) (color 0 0 0 0)
+  )
   (junction (at 160.02 76.2) (diameter 0) (color 0 0 0 0)
   )
@@
   )
   (junction (at 88.9 99.06) (diameter 0) (color 0 0 0 0)
-  )
-  (junction (at 160.02 25.4) (diameter 0) (color 0 0 0 0)
   )
   (junction (at 114.3 99.06) (diameter 0) (color 0 0 0 0)
@@
     (stroke (width 0) (type default) (color 0 0 0 0))
   )
+  (wire (pts (xy 100.33 25.4) (xy 107.95 25.4))
+    (stroke (width 0) (type default) (color 0 0 0 0))
+  )
   (wire (pts (xy 138.43 78.74) (xy 138.43 76.2))
     (stroke (width 0) (type default) (color 0 0 0 0))
@@
     (stroke (width 0) (type default) (color 0 0 0 0))
   )
+  (wire (pts (xy 100.33 22.86) (xy 100.33 25.4))
+    (stroke (width 0) (type default) (color 0 0 0 0))
+  )
   (wire (pts (xy 63.5 129.54) (xy 63.5 132.08))
     (stroke (width 0) (type default) (color 0 0 0 0))
@@
     (stroke (width 0) (type default) (color 0 0 0 0))
   )
-  (wire (pts (xy 121.92 22.86) (xy 121.92 25.4))
+  (wire (pts (xy 118.11 25.4) (xy 121.92 25.4))
     (stroke (width 0) (type default) (color 0 0 0 0))
   )
@@
     (stroke (width 0) (type default) (color 0 0 0 0))
   )
+  (wire (pts (xy 107.95 25.4) (xy 110.49 25.4))
+    (stroke (width 0) (type default) (color 0 0 0 0))
+  )
   (wire (pts (xy 114.3 129.54) (xy 139.7 129.54))
     (stroke (width 0) (type default) (color 0 0 0 0))
@@
     (stroke (width 0) (type default) (color 0 0 0 0))
   )
-  (label "5V" (at 152.4 25.4 0)
+  (wire (pts (xy 107.95 22.86) (xy 107.95 25.4))
+    (stroke (width 0) (type default) (color 0 0 0 0))
+  )
+  (label "5V_EMITTERS" (at 142.24 25.4 0)
     (effects (font (size 1.27 1.27)) (justify left bottom))
   )
   (label "EMITTER_K" (at 121.92 54.61 0)
     (effects (font (size 1.27 1.27)) (justify left bottom))
-  )
-  (label "D12_EMITTERS" (at 96.52 60.96 180)
-    (effects (font (size 1.27 1.27)) (justify right bottom))
   )
   (global_label "D6_LED_RIGHT" (shape input) (at 102.87 171.45 180) (fields_autoplaced)
@@
     )
   )
+  (global_label "5V" (shape input) (at 100.33 25.4 180) (fields_autoplaced)
+    (effects (font (size 1.27 1.27)) (justify right))
+    (property "Intersheet References" "${INTERSHEET_REFS}" (id 0) (at 95.6188 25.3206 0)
+      (effects (font (size 1.27 1.27)) (justify right) hide)
+    )
+  )
   (global_label "D11_LED_LEFT" (shape input) (at 102.87 163.83 180) (fields_autoplaced)
     (effects (font (size 1.27 1.27)) (justify right))
@@
     )
   )
+  (global_label "D12_EMITTERS" (shape input) (at 90.17 60.96 180) (fields_autoplaced)
+    (effects (font (size 1.27 1.27)) (justify right))
+    (property "Intersheet References" "${INTERSHEET_REFS}" (id 0) (at 74.3312 61.0394 0)
+      (effects (font (size 1.27 1.27)) (justify right) hide)
+    )
+  )
   (global_label "D12_EMITTERS" (shape input) (at 46.99 49.53 0) (fields_autoplaced)
     (effects (font (size 1.27 1.27)) (justify left))
@@
     (pin "2")
   )
-  (symbol (lib_id "power:PWR_FLAG") (at 160.02 25.4 0) (unit 1)
-    (in_bom yes) (on_board yes) (fields_autoplaced)
-    (property "Reference" "#FLG01" (id 0) (at 160.02 23.495 0)
-      (effects (font (size 1.27 1.27)) hide)
-    )
-    (property "Value" "PWR_FLAG" (id 1) (at 160.02 21.8242 0))
-    (property "Footprint" "" (id 2) (at 160.02 25.4 0)
-      (effects (font (size 1.27 1.27)) hide)
-    )
-    (property "Datasheet" "~" (id 3) (at 160.02 25.4 0)
-      (effects (font (size 1.27 1.27)) hide)
-    )
-    (pin "1")
-  )
-  (symbol (lib_id "power:+5V") (at 121.92 22.86 0) (unit 1)
-    (in_bom yes) (on_board yes) (fields_autoplaced)
-    (property "Reference" "#PWR01" (id 0) (at 121.92 26.67 0)
-      (effects (font (size 1.27 1.27)) hide)
-    )
-    (property "Value" "+5V" (id 1) (at 121.92 19.2842 0))
-    (property "Footprint" "" (id 2) (at 121.92 22.86 0)
-      (effects (font (size 1.27 1.27)) hide)
-    )
-    (property "Datasheet" "" (id 3) (at 121.92 22.86 0)
+  (symbol (lib_id "Device:R") (at 114.3 25.4 270) (unit 1)
+    (in_bom yes) (on_board yes)
+    (property "Reference" "R12" (id 0) (at 114.3 22.86 90))
+    (property "Value" "33R" (id 1) (at 114.3 25.4 90))
+    (property "Footprint" "Resistor_THT:R_Axial_DIN0207_L6.3mm_D2.5mm_P7.62mm_Horizontal" (id 2) (at 114.3 23.622 90)
+      (effects (font (size 1.27 1.27)) hide)
+    )
+    (property "Datasheet" "~" (id 3) (at 114.3 25.4 0)
+      (effects (font (size 1.27 1.27)) hide)
+    )
+    (pin "1")
+    (pin "2")
+  )
+  (symbol (lib_id "power:PWR_FLAG") (at 100.33 22.86 0) (unit 1)
+    (in_bom yes) (on_board yes) (fields_autoplaced)
+    (property "Reference" "#FLG01" (id 0) (at 100.33 20.955 0)
+      (effects (font (size 1.27 1.27)) hide)
+    )
+    (property "Value" "PWR_FLAG" (id 1) (at 100.33 19.2842 0))
+    (property "Footprint" "" (id 2) (at 100.33 22.86 0)
+      (effects (font (size 1.27 1.27)) hide)
+    )
+    (property "Datasheet" "~" (id 3) (at 100.33 22.86 0)
+      (effects (font (size 1.27 1.27)) hide)
+    )
+    (pin "1")
+  )
+  (symbol (lib_id "power:+5V") (at 107.95 22.86 0) (unit 1)
+    (in_bom yes) (on_board yes) (fields_autoplaced)
+    (property "Reference" "#PWR01" (id 0) (at 107.95 26.67 0)
+      (effects (font (size 1.27 1.27)) hide)
+    )
+    (property "Value" "+5V" (id 1) (at 107.95 19.2842 0))
+    (property "Footprint" "" (id 2) (at 107.95 22.86 0)
+      (effects (font (size 1.27 1.27)) hide)
+    )
+    (property "Datasheet" "" (id 3) (at 107.95 22.86 0)
       (effects (font (size 1.27 1.27)) hide)
     )
@@
       (reference "R11") (unit 1) (value "2k0") (footprint "Resistor_THT:R_Axial_DIN0207_L6.3mm_D2.5mm_P7.62mm_Horizontal")
     )
-  )
+    (path "/5e1a1e58-91b2-4813-89b0-9363148b64b4"
+      (reference "R12") (unit 1) (value "33R") (footprint "Resistor_THT:R_Axial_DIN0207_L6.3mm_D2.5mm_P7.62mm_Horizontal")
+    )
+  )
