File: kicad/line-sensor-mini-wide/line-sensor-mini-wide.kicad_pcb (KiCad board)
At the start: 2 copper layers, 28.7 x 81.3 mm, 37 parts, among them J1 SENSORS, Q1 BC337, Q2 BC337, Q3 BPW85C, Q4 BPW85C, Q5 BPW85C, Q6 BPW85C, Q7 BPW85C, Q8 BPW85C

Commit message: update for line-sensor-mini-wide v1.0
Other:
- board text added: "3V3"
- board text added: "5V"
- board text added: "A0"
- board text added: "A1"
- board text added: "A2"
- board text added: "A3"
- board text added: "A4"
- board text added: "A5"
- board text added: "D11"
- board text added: "D12"
- board text added: "D6"
- board text added: "GND"
Changed lines of the file:
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@@
     (effects (font (size 1.5 1.5) (thickness 0.3)) (justify mirror))
+  )
+  (gr_text "5V" (at 143.1 118.97) (layer "F.SilkS")
+    (effects (font (size 1 1) (thickness 0.15)) (justify left))
+  )
+  (gr_text "A3" (at 143.1 98.65) (layer "F.SilkS")
+    (effects (font (size 1 1) (thickness 0.15)) (justify left))
   )
   (gr_text "LINE SENSOR MINI" (at 140 125.5 90) (layer "F.SilkS")
@@
     (effects (font (size 1 1) (thickness 0.15)))
   )
+  (gr_text "3V3" (at 143.1 121.51) (layer "F.SilkS")
+    (effects (font (size 1 1) (thickness 0.15)) (justify left))
+  )
   (gr_text "c" (at 150.75 131.75) (layer "F.SilkS")
     (effects (font (size 1 1) (thickness 0.15)))
+  )
+  (gr_text "D6" (at 143.1 113.89) (layer "F.SilkS")
+    (effects (font (size 1 1) (thickness 0.15)) (justify left))
+  )
+  (gr_text "A0" (at 143.1 106.27) (layer "F.SilkS")
+    (effects (font (size 1 1) (thickness 0.15)) (justify left))
   )
   (gr_text "e" (at 150.75 126) (layer "F.SilkS")
     (effects (font (size 1 1) (thickness 0.15)))
   )
+  (gr_text "GND" (at 143.1 91.03) (layer "F.SilkS")
+    (effects (font (size 1 1) (thickness 0.15)) (justify left))
+  )
   (gr_text "V1.0" (at 140 114.5 90) (layer "F.SilkS")
     (effects (font (size 1 1) (thickness 0.15)))
   )
+  (gr_text "A4" (at 143.1 96.11) (layer "F.SilkS")
+    (effects (font (size 1 1) (thickness 0.15)) (justify left))
+  )
+  (gr_text "D11" (at 143.1 108.81) (layer "F.SilkS")
+    (effects (font (size 1 1) (thickness 0.15)) (justify left))
+  )
+  (gr_text "GND" (at 143.1 116.43) (layer "F.SilkS")
+    (effects (font (size 1 1) (thickness 0.15)) (justify left))
+  )
   (gr_text "UKMARSBOT" (at 140 81 90) (layer "F.SilkS")
     (effects (font (size 1.25 1.25) (thickness 0.2)))
+  )
+  (gr_text "A2" (at 143.1 101.19) (layer "F.SilkS")
+    (effects (font (size 1 1) (thickness 0.15)) (justify left))
+  )
+  (gr_text "A1" (at 143.1 103.73) (layer "F.SilkS")
+    (effects (font (size 1 1) (thickness 0.15)) (justify left))
+  )
+  (gr_text "A5" (at 143.1 93.57) (layer "F.SilkS")
+    (effects (font (size 1 1) (thickness 0.15)) (justify left))
+  )
+  (gr_text "5V" (at 143.1 88.49) (layer "F.SilkS")
+    (effects (font (size 1 1) (thickness 0.15)) (justify left))
+  )
+  (gr_text "D12" (at 143.1 111.35) (layer "F.SilkS")
+    (effects (font (size 1 1) (thickness 0.15)) (justify left))
   )
   (gr_text "e" (at 150.25 78) (layer "F.SilkS")
@@
   (segment (start 154.01548 144.75) (end 143.5 144.75) (width 0.75) (layer "F.Cu") (net 5))
   (segment (start 150 110) (end 150 110.7) (width 0.5) (layer "F.Cu") (net 5))
+  (segment (start 142 88.49) (end 146.47 88.49) (width 1.25) (layer "F.Cu") (net 5))
   (segment (start 166.444031 77.818756) (end 157.187638 68.562362) (width 0.75) (layer "F.Cu") (net 5))
   (segment (start 150 100) (end 154.1 95.9) (width 0.5) (layer "F.Cu") (net 5))
@@
   (segment (start 151.169031 123.194031) (end 166.444031 123.194031) (width 0.5) (layer "F.Cu") (net 5))
   (segment (start 156.3 117) (end 161.352233 117) (width 0.5) (layer "F.Cu") (net 5))
+  (segment (start 149.73 88.25) (end 157 88.25) (width 1.25) (layer "F.Cu") (net 5))
   (segment (start 154.1 95.9) (end 158 95.9) (width 0.5) (layer "F.Cu") (net 5))
   (segment (start 166.444031 119.805969) (end 166.444031 120.055969) (width 0.75) (layer "F.Cu") (net 5))
@@
   (segment (start 158.9 90.15) (end 157 88.25) (width 0.5) (layer "F.Cu") (net 5))
   (segment (start 154.62 71) (end 157.057638 68.562362) (width 0.75) (layer "F.Cu") (net 5))
+  (segment (start 146.47 88.49) (end 147.98 90) (width 1.25) (layer "F.Cu") (net 5))
   (segment (start 158.9 95) (end 158.9 90.15) (width 0.5) (layer "F.Cu") (net 5))
   (segment (start 158 95.9) (end 158.9 95) (width 0.5) (layer "F.Cu") (net 5))
   (segment (start 157.12774 141.50774) (end 157.25774 141.50774) (width 0.75) (layer "F.Cu") (net 5))
   (segment (start 157.25774 141.50774) (end 154.01548 144.75) (width 0.75) (layer "F.Cu") (net 5))
+  (segment (start 147.98 90) (end 149.73 88.25) (width 1.25) (layer "F.Cu") (net 5))
   (segment (start 143.5 65.25) (end 140.75 68) (width 0.75) (layer "F.Cu") (net 5))
   (segment (start 154.62 139) (end 157.12774 141.50774) (width 0.75) (layer "F.Cu") (net 5))
   (segment (start 157.057638 68.562362) (end 157.187638 68.562362) (width 0.75) (layer "F.Cu") (net 5))
   (segment (start 161.352233 117) (end 164.408202 120.055969) (width 0.5) (layer "F.Cu") (net 5))
-  (segment (start 147.975 90) (end 149.725 88.25) (width 0.75) (layer "B.Cu") (net 5))
-  (segment (start 149.725 88.25) (end 157 88.25) (width 0.75) (layer "B.Cu") (net 5))
-  (segment (start 146.465 88.49) (end 147.975 90) (width 0.75) (layer "B.Cu") (net 5))
-  (segment (start 142 88.49) (end 146.465 88.49) (width 0.75) (layer "B.Cu") (net 5))
   (segment (start 143.410756 134.65) (end 159.19 134.65) (width 0.5) (layer "F.Cu") (net 6))
   (segment (start 139.800499 131.039743) (end 143.410756 134.65) (width 0.5) (layer "F.Cu") (net 6))
@@
   (segment (start 139.4 71.89) (end 139.4 90.97) (width 0.5) (layer "F.Cu") (net 9))
   (segment (start 139.4 90.97) (end 142 93.57) (width 0.5) (layer "F.Cu") (net 9))
-  (segment (start 142 96.11) (end 144.405 96.11) (width 0.5) (layer "F.Cu") (net 10))
-  (segment (start 144.405 96.11) (end 150.515 90) (width 0.5) (layer "F.Cu") (net 10))
-  (segment (start 150.515 90) (end 155.75 90) (width 0.5) (layer "F.Cu") (net 10))
+  (segment (start 150.52 90) (end 155.75 90) (width 0.5) (layer "F.Cu") (net 10))
+  (segment (start 142 96.11) (end 144.41 96.11) (width 0.5) (layer "F.Cu") (net 10))
   (segment (start 155.75 90) (end 157 91.25) (width 0.5) (layer "F.Cu") (net 10))
+  (segment (start 144.41 96.11) (end 150.52 90) (width 0.5) (layer "F.Cu") (net 10))
   (segment (start 157.13 129.94) (end 157.19 130) (width 0.5) (layer "F.Cu") (net 11))
   (segment (start 157.13 127) (end 157.13 129.94) (width 0.5) (layer "F.Cu") (net 11))
@@
   (segment (start 148.3 103.3) (end 150 105) (width 0.5) (layer "F.Cu") (net 12))
   (segment (start 146 125.18) (end 152.36 131.54) (width 0.5) (layer "F.Cu") (net 12))
-  (segment (start 140.75 83) (end 142 84.25) (width 0.5) (layer "F.Cu") (net 13))
-  (segment (start 149.25 84.25) (end 149.96 83.54) (width 0.5) (layer "F.Cu") (net 13))
+  (segment (start 140.75 83) (end 142.35 84.6) (width 0.5) (layer "F.Cu") (net 13))
+  (segment (start 150.94 84.6) (end 152 83.54) (width 0.5) (layer "F.Cu") (net 13))
+  (segment (start 142.35 84.6) (end 150.94 84.6) (width 0.5) (layer "F.Cu") (net 13))
   (segment (start 140.75 74) (end 140.75 83) (width 0.5) (layer "F.Cu") (net 13))
-  (segment (start 142 84.25) (end 149.25 84.25) (width 0.5) (layer "F.Cu") (net 13))
-  (segment (start 149.96 83.54) (end 152 83.54) (width 0.5) (layer "F.Cu") (net 13))
   (segment (start 140.75 74) (end 139.153 75.597) (width 0.75) (layer "B.Cu") (net 13))
   (segment (start 139.153 75.597) (end 139.153 134.403) (width 0.75) (layer "B.Cu") (net 13))
