File: ecad/kicad/line-sensor-mini-wide/line-sensor-mini-wide.kicad_sch (KiCad schematic)
At the start: 37 parts, among them J1 SENSORS, Q1 BC337, Q2 BC337, Q3 BPW85C, Q4 BPW85C, Q5 BPW85C, Q6 BPW85C, Q7 BPW85C, Q8 BPW85C

Commit message: improve BOM for mini wide line sensor
Parts:
- C1: Note (none) -> 16V, 10mm Dia. Electrolytic; Package (none) -> Axial Lead, 0.1" or 0.2"
- D1, D2, D3, D4, D5: Note (none) -> IR or visible sensor emitter
- D6, D7: Note (none) -> 3mm Indicator LED
- H1, H2: Package 3.2mm hole -> M3 clearance, 3.2mm; now left out of the parts list
- J1: Note (none) -> Pin Header, socket on sensor board
- Q1, Q2: Note (none) -> 0.8A NPN or FET
- Q3, Q4, Q5, Q6, Q7, Q8: Note (none) -> Must be matched to emitters
- R1, R10, R11, R12, R13, R14, R15, R16, R2, R26, R27, R3, R4, R5, R6, R7, R8, R9: Note (none) -> ¼W or ⅛W, 5% or 10%, carbon or metal film
Changed lines of the file:
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@@
+      (effects (font (size 1.27 1.27)) hide)
+    )
+    (property "Note" "¼W or ⅛W, 5% or 10%, carbon or metal film" (id 5) (at 114.3 123.19 0)
       (effects (font (size 1.27 1.27)) hide)
     )
@@
       (effects (font (size 1.27 1.27)) hide)
     )
+    (property "Note" "¼W or ⅛W, 5% or 10%, carbon or metal film" (id 5) (at 236.22 59.69 0)
+      (effects (font (size 1.27 1.27)) hide)
+    )
     (pin "1")
     (pin "2")
@@
       (effects (font (size 1.27 1.27)) hide)
     )
+    (property "Note" "3mm Indicator LED" (id 5) (at 91.44 153.67 0)
+      (effects (font (size 1.27 1.27)) hide)
+    )
     (pin "1")
     (pin "2")
@@
       (effects (font (size 1.27 1.27)) hide)
     )
+    (property "Note" "¼W or ⅛W, 5% or 10%, carbon or metal film" (id 5) (at 121.92 31.75 0)
+      (effects (font (size 1.27 1.27)) hide)
+    )
     (pin "1")
     (pin "2")
@@
     )
     (property "Datasheet" "~" (id 3) (at 160.02 43.18 0)
+      (effects (font (size 1.27 1.27)) hide)
+    )
+    (property "Package" "Axial Lead, 0.1\" or 0.2\"" (id 4) (at 160.02 43.18 0)
+      (effects (font (size 1.27 1.27)) hide)
+    )
+    (property "Note" "16V, 10mm Dia. Electrolytic" (id 5) (at 160.02 43.18 0)
       (effects (font (size 1.27 1.27)) hide)
     )
@@
       (effects (font (size 1.27 1.27)) hide)
     )
+    (property "Note" "¼W or ⅛W, 5% or 10%, carbon or metal film" (id 5) (at 149.86 31.75 0)
+      (effects (font (size 1.27 1.27)) hide)
+    )
     (pin "1")
     (pin "2")
@@
       (effects (font (size 1.27 1.27)) hide)
     )
+    (property "Note" "¼W or ⅛W, 5% or 10%, carbon or metal film" (id 5) (at 102.87 153.67 0)
+      (effects (font (size 1.27 1.27)) hide)
+    )
     (pin "1")
     (pin "2")
@@
     )
     (property "Package" "TO92" (id 4) (at 119.38 60.96 0)
+      (effects (font (size 1.27 1.27)) hide)
+    )
+    (property "Note" "0.8A NPN or FET" (id 5) (at 119.38 60.96 0)
       (effects (font (size 1.27 1.27)) hide)
     )
@@
       (effects (font (size 1.27 1.27)) hide)
     )
+    (property "Note" "IR or visible sensor emitter" (id 5) (at 135.89 43.18 0)
+      (effects (font (size 1.27 1.27)) hide)
+    )
     (pin "1")
     (pin "2")
@@
     )
     (property "Package" "T-1 (3mm)" (id 4) (at 137.16 106.68 0)
+      (effects (font (size 1.27 1.27)) hide)
+    )
+    (property "Note" "Must be matched to emitters" (id 5) (at 137.16 106.68 0)
       (effects (font (size 1.27 1.27)) hide)
     )
@@
       (effects (font (size 1.27 1.27)) hide)
     )
+    (property "Note" "¼W or ⅛W, 5% or 10%, carbon or metal film" (id 5) (at 63.5 123.19 0)
+      (effects (font (size 1.27 1.27)) hide)
+    )
     (pin "1")
     (pin "2")
@@
       (effects (font (size 1.27 1.27)) hide)
     )
+    (property "Note" "¼W or ⅛W, 5% or 10%, carbon or metal film" (id 5) (at 243.84 67.31 0)
+      (effects (font (size 1.27 1.27)) hide)
+    )
     (pin "1")
     (pin "2")
@@
     )
     (property "Package" "T-1 (3mm)" (id 4) (at 121.92 43.18 0)
+      (effects (font (size 1.27 1.27)) hide)
+    )
+    (property "Note" "IR or visible sensor emitter" (id 5) (at 121.92 43.18 0)
       (effects (font (size 1.27 1.27)) hide)
     )
@@
       (effects (font (size 1.27 1.27)) hide)
     )
+    (property "Note" "¼W or ⅛W, 5% or 10%, carbon or metal film " (id 5) (at 114.3 25.4 0)
+      (effects (font (size 1.27 1.27)) hide)
+    )
     (pin "1")
     (pin "2")
@@
     )
     (property "Package" "T-1 (3mm)" (id 4) (at 86.36 106.68 0)
+      (effects (font (size 1.27 1.27)) hide)
+    )
+    (property "Note" "Must be matched to emitters" (id 5) (at 86.36 106.68 0)
       (effects (font (size 1.27 1.27)) hide)
     )
@@
       (effects (font (size 1.27 1.27)) hide)
     )
+    (property "Note" "¼W or ⅛W, 5% or 10%, carbon or metal film" (id 5) (at 255.27 30.48 0)
+      (effects (font (size 1.27 1.27)) hide)
+    )
     (pin "1")
     (pin "2")
@@
     )
     (property "Package" "14 pin 0.1\" header" (id 4) (at 31.75 44.45 0)
+      (effects (font (size 1.27 1.27)) hide)
+    )
+    (property "Note" "Pin Header, socket on sensor board" (id 5) (at 31.75 44.45 0)
       (effects (font (size 1.27 1.27)) hide)
     )
@@
       (effects (font (size 1.27 1.27)) hide)
     )
+    (property "Note" "Must be matched to emitters" (id 5) (at 162.56 106.68 0)
+      (effects (font (size 1.27 1.27)) hide)
+    )
     (pin "1")
     (pin "2")
   )
   (symbol (lib_id "Mechanical:MountingHole") (at 35.56 172.72 0) (unit 1)
-    (in_bom yes) (on_board yes)
+    (in_bom no) (on_board yes)
     (property "Reference" "H2" (id 0) (at 39.37 172.72 0))
     (property "Value" "MountingHole" (id 1) (at 35.56 169.545 0)
@@
       (effects (font (size 1.27 1.27)) hide)
     )
-    (property "Package" "3.2mm hole" (id 4) (at 35.56 172.72 0)
+    (property "Package" "M3 clearance, 3.2mm" (id 4) (at 35.56 172.72 0)
       (effects (font (size 1.27 1.27)) hide)
     )
@@
       (effects (font (size 1.27 1.27)) hide)
     )
+    (property "Note" "¼W or ⅛W, 5% or 10%, carbon or metal film" (id 5) (at 135.89 31.75 0)
+      (effects (font (size 1.27 1.27)) hide)
+    )
     (pin "1")
     (pin "2")
@@
       (effects (font (size 1.27 1.27)) hide)
     )
+    (property "Note" "¼W or ⅛W, 5% or 10%, carbon or metal film" (id 5) (at 269.24 30.48 0)
+      (effects (font (size 1.27 1.27)) hide)
+    )
     (pin "1")
     (pin "2")
@@
       (effects (font (size 1.27 1.27)) hide)
     )
+    (property "Note" "¼W or ⅛W, 5% or 10%, carbon or metal film" (id 5) (at 102.87 163.83 0)
+      (effects (font (size 1.27 1.27)) hide)
+    )
     (pin "1")
     (pin "2")
@@
     )
     (property "Package" "TO92" (id 4) (at 252.73 59.69 0)
+      (effects (font (size 1.27 1.27)) hide)
+    )
+    (property "Note" "0.8A NPN or FET" (id 5) (at 252.73 59.69 0)
       (effects (font (size 1.27 1.27)) hide)
     )
@@
       (effects (font (size 1.27 1.27)) hide)
     )
+    (property "Note" "¼W or ⅛W, 5% or 10%, carbon or metal film" (id 5) (at 88.9 123.19 0)
+      (effects (font (size 1.27 1.27)) hide)
+    )
     (pin "1")
     (pin "2")
@@
       (effects (font (size 1.27 1.27)) hide)
     )
+    (property "Note" "IR or visible sensor emitter" (id 5) (at 269.24 41.91 0)
+      (effects (font (size 1.27 1.27)) hide)
+    )
     (pin "1")
     (pin "2")
@@
       (effects (font (size 1.27 1.27)) hide)
     )
+    (property "Note" "Must be matched to emitters" (id 5) (at 60.96 106.68 0)
+      (effects (font (size 1.27 1.27)) hide)
+    )
     (pin "1")
     (pin "2")
   )
   (symbol (lib_id "Mechanical:MountingHole") (at 35.56 165.1 0) (unit 1)
-    (in_bom yes) (on_board yes) (fields_autoplaced)
+    (in_bom no) (on_board yes) (fields_autoplaced)
     (property "Reference" "H1" (id 0) (at 38.1 164.2653 0)
       (effects (font (size 1.27 1.27)) (justify left))
@@
       (effects (font (size 1.27 1.27)) hide)
     )
-    (property "Package" "3.2mm hole" (id 4) (at 35.56 165.1 0)
+    (property "Package" "M3 clearance, 3.2mm" (id 4) (at 35.56 165.1 0)
       (effects (font (size 1.27 1.27)) hide)
     )
@@
       (effects (font (size 1.27 1.27)) hide)
     )
+    (property "Note" "¼W or ⅛W, 5% or 10%, carbon or metal film" (id 5) (at 102.87 60.96 0)
+      (effects (font (size 1.27 1.27)) hide)
+    )
     (pin "1")
     (pin "2")
@@
       (effects (font (size 1.27 1.27)) hide)
     )
+    (property "Note" "¼W or ⅛W, 5% or 10%, carbon or metal film" (id 5) (at 110.49 68.58 0)
+      (effects (font (size 1.27 1.27)) hide)
+    )
     (pin "1")
     (pin "2")
@@
     )
     (property "Package" "T-1 (3mm)" (id 4) (at 111.76 106.68 0)
+      (effects (font (size 1.27 1.27)) hide)
+    )
+    (property "Note" "Must be matched to emitters" (id 5) (at 111.76 106.68 0)
       (effects (font (size 1.27 1.27)) hide)
     )
@@
       (effects (font (size 1.27 1.27)) hide)
     )
+    (property "Note" "¼W or ⅛W, 5% or 10%, carbon or metal film" (id 5) (at 139.7 123.19 0)
+      (effects (font (size 1.27 1.27)) hide)
+    )
     (pin "1")
     (pin "2")
@@
       (effects (font (size 1.27 1.27)) hide)
     )
+    (property "Note" "3mm Indicator LED" (id 5) (at 91.44 163.83 0)
+      (effects (font (size 1.27 1.27)) hide)
+    )
     (pin "1")
     (pin "2")
@@
     )
     (property "Package" "T-1 (3mm)" (id 4) (at 187.96 106.68 0)
+      (effects (font (size 1.27 1.27)) hide)
+    )
+    (property "Note" "Must be matched to emitters" (id 5) (at 187.96 106.68 0)
       (effects (font (size 1.27 1.27)) hide)
     )
@@
     )
     (property "Package" "T-1 (3mm)" (id 4) (at 255.27 41.91 0)
+      (effects (font (size 1.27 1.27)) hide)
+    )
+    (property "Note" "IR or visible sensor emitter" (id 5) (at 255.27 41.91 0)
       (effects (font (size 1.27 1.27)) hide)
     )
@@
       (effects (font (size 1.27 1.27)) hide)
     )
+    (property "Note" "¼W or ⅛W, 5% or 10%, carbon or metal film" (id 5) (at 165.1 123.19 0)
+      (effects (font (size 1.27 1.27)) hide)
+    )
     (pin "1")
     (pin "2")
@@
       (effects (font (size 1.27 1.27)) hide)
     )
+    (property "Note" "IR or visible sensor emitter" (id 5) (at 149.86 43.18 0)
+      (effects (font (size 1.27 1.27)) hide)
+    )
     (pin "1")
     (pin "2")
@@
       (effects (font (size 1.27 1.27)) hide)
     )
+    (property "Note" "¼W or ⅛W, 5% or 10%, carbon or metal film" (id 5) (at 190.5 123.19 0)
+      (effects (font (size 1.27 1.27)) hide)
+    )
