File: ecad/kicad/mainboard/mainboard.kicad_sch (KiCad schematic)
At the start: 34 parts, among them IC1 74HC86, J1 SENSORS, J2 CONN_06SILK_FEMALE_PTH, J3 CONN_06SILK_FEMALE_PTH, J4 POWER, J5 SERIAL, M1 Left Motor, M2 Right Motor, U1 Arduino_Nano, U2 TB6612FNG-Module

Commit message: re-route kicad mainboard with bigger pads
Parts:
- R1, R10, R11, R2, R3, R4, R5, R6, R7, R8: footprint ukmarsbot:R_Axial_DIN0207_L6.3mm_D2.5mm_P7.62mm_Horizontal -> ukmarsbot:R_Axial_DIN0207_L6.3mm_D2.5mm_P7.62mm_BIGPAD
Changed lines of the file:
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@@
     (property "Reference" "R10" (id 0) (at 50.8 29.21 0))
     (property "Value" "10k" (id 1) (at 50.8 33.02 0))
-    (property "Footprint" "ukmarsbot:R_Axial_DIN0207_L6.3mm_D2.5mm_P7.62mm_Horizontal" (id 2) (at 45.212 31.75 90)
+    (property "Footprint" "ukmarsbot:R_Axial_DIN0207_L6.3mm_D2.5mm_P7.62mm_BIGPAD" (id 2) (at 45.212 31.75 90)
       (effects (font (size 1.27 1.27)) hide)
     )
@@
       (effects (font (size 1.75 1.75)) (justify right top))
     )
-    (property "Footprint" "ukmarsbot:R_Axial_DIN0207_L6.3mm_D2.5mm_P7.62mm_Horizontal" (id 2) (at 165.1 150.368 90)
+    (property "Footprint" "ukmarsbot:R_Axial_DIN0207_L6.3mm_D2.5mm_P7.62mm_BIGPAD" (id 2) (at 165.1 150.368 90)
       (effects (font (size 1.27 1.27)) hide)
     )
@@
       (effects (font (size 1.75 1.75)) (justify right top))
     )
-    (property "Footprint" "ukmarsbot:R_Axial_DIN0207_L6.3mm_D2.5mm_P7.62mm_Horizontal" (id 2) (at 255.778 48.26 90)
+    (property "Footprint" "ukmarsbot:R_Axial_DIN0207_L6.3mm_D2.5mm_P7.62mm_BIGPAD" (id 2) (at 255.778 48.26 90)
       (effects (font (size 1.27 1.27)) hide)
     )
@@
     (property "Reference" "R11" (id 0) (at 54.61 14.3342 90))
     (property "Value" "4k7" (id 1) (at 54.61 16.8711 90))
-    (property "Footprint" "ukmarsbot:R_Axial_DIN0207_L6.3mm_D2.5mm_P7.62mm_Horizontal" (id 2) (at 54.61 20.828 90)
+    (property "Footprint" "ukmarsbot:R_Axial_DIN0207_L6.3mm_D2.5mm_P7.62mm_BIGPAD" (id 2) (at 54.61 20.828 90)
       (effects (font (size 1.27 1.27)) hide)
     )
@@
       (effects (font (size 1.75 1.75)) (justify right top))
     )
-    (property "Footprint" "ukmarsbot:R_Axial_DIN0207_L6.3mm_D2.5mm_P7.62mm_Horizontal" (id 2) (at 174.498 156.21 90)
+    (property "Footprint" "ukmarsbot:R_Axial_DIN0207_L6.3mm_D2.5mm_P7.62mm_BIGPAD" (id 2) (at 174.498 156.21 90)
       (effects (font (size 1.27 1.27)) hide)
     )
@@
       (effects (font (size 1.75 1.75)) (justify left bottom))
     )
-    (property "Footprint" "ukmarsbot:R_Axial_DIN0207_L6.3mm_D2.5mm_P7.62mm_Horizontal" (id 2) (at 119.38 146.812 90)
+    (property "Footprint" "ukmarsbot:R_Axial_DIN0207_L6.3mm_D2.5mm_P7.62mm_BIGPAD" (id 2) (at 119.38 146.812 90)
       (effects (font (size 1.27 1.27)) hide)
     )
@@
       (effects (font (size 1.75 1.75)) (justify right top))
     )
-    (property "Footprint" "ukmarsbot:R_Axial_DIN0207_L6.3mm_D2.5mm_P7.62mm_Horizontal" (id 2) (at 105.918 133.35 90)
+    (property "Footprint" "ukmarsbot:R_Axial_DIN0207_L6.3mm_D2.5mm_P7.62mm_BIGPAD" (id 2) (at 105.918 133.35 90)
       (effects (font (size 1.27 1.27)) hide)
     )
@@
       (effects (font (size 1.75 1.75)) (justify right top))
     )
-    (property "Footprint" "ukmarsbot:R_Axial_DIN0207_L6.3mm_D2.5mm_P7.62mm_Horizontal" (id 2) (at 255.778 66.04 90)
+    (property "Footprint" "ukmarsbot:R_Axial_DIN0207_L6.3mm_D2.5mm_P7.62mm_BIGPAD" (id 2) (at 255.778 66.04 90)
       (effects (font (size 1.27 1.27)) hide)
     )
@@
       (effects (font (size 1.75 1.75)) (justify left bottom))
     )
-    (property "Footprint" "ukmarsbot:R_Axial_DIN0207_L6.3mm_D2.5mm_P7.62mm_Horizontal" (id 2) (at 135.89 146.812 90)
+    (property "Footprint" "ukmarsbot:R_Axial_DIN0207_L6.3mm_D2.5mm_P7.62mm_BIGPAD" (id 2) (at 135.89 146.812 90)
       (effects (font (size 1.27 1.27)) hide)
     )
@@
       (effects (font (size 1.75 1.75)) (justify left bottom))
     )
-    (property "Footprint" "ukmarsbot:R_Axial_DIN0207_L6.3mm_D2.5mm_P7.62mm_Horizontal" (id 2) (at 151.13 146.812 90)
+    (property "Footprint" "ukmarsbot:R_Axial_DIN0207_L6.3mm_D2.5mm_P7.62mm_BIGPAD" (id 2) (at 151.13 146.812 90)
       (effects (font (size 1.27 1.27)) hide)
     )
@@
     )
     (path "/5e6a31d8-da64-439f-970e-591de48617a0"
-      (reference "R1") (unit 1) (value "10k") (footprint "ukmarsbot:R_Axial_DIN0207_L6.3mm_D2.5mm_P7.62mm_Horizontal")
+      (reference "R1") (unit 1) (value "10k") (footprint "ukmarsbot:R_Axial_DIN0207_L6.3mm_D2.5mm_P7.62mm_BIGPAD")
     )
     (path "/412dd346-5075-4419-be0d-bf3f31c29907"
-      (reference "R2") (unit 1) (value "10k") (footprint "ukmarsbot:R_Axial_DIN0207_L6.3mm_D2.5mm_P7.62mm_Horizontal")
+      (reference "R2") (unit 1) (value "10k") (footprint "ukmarsbot:R_Axial_DIN0207_L6.3mm_D2.5mm_P7.62mm_BIGPAD")
     )
     (path "/8290c828-8e38-4225-be08-a8af654d7bdd"
-      (reference "R3") (unit 1) (value "4k7") (footprint "ukmarsbot:R_Axial_DIN0207_L6.3mm_D2.5mm_P7.62mm_Horizontal")
+      (reference "R3") (unit 1) (value "4k7") (footprint "ukmarsbot:R_Axial_DIN0207_L6.3mm_D2.5mm_P7.62mm_BIGPAD")
     )
     (path "/d88df602-0039-4964-be9e-02ef1bde45d4"
-      (reference "R4") (unit 1) (value "2k2") (footprint "ukmarsbot:R_Axial_DIN0207_L6.3mm_D2.5mm_P7.62mm_Horizontal")
+      (reference "R4") (unit 1) (value "2k2") (footprint "ukmarsbot:R_Axial_DIN0207_L6.3mm_D2.5mm_P7.62mm_BIGPAD")
     )
     (path "/12bf2296-306d-483a-86da-45d5850ec863"
-      (reference "R5") (unit 1) (value "1k0") (footprint "ukmarsbot:R_Axial_DIN0207_L6.3mm_D2.5mm_P7.62mm_Horizontal")
+      (reference "R5") (unit 1) (value "1k0") (footprint "ukmarsbot:R_Axial_DIN0207_L6.3mm_D2.5mm_P7.62mm_BIGPAD")
     )
     (path "/410c1284-b5db-4d53-9744-6756a777d596"
-      (reference "R6") (unit 1) (value "470") (footprint "ukmarsbot:R_Axial_DIN0207_L6.3mm_D2.5mm_P7.62mm_Horizontal")
+      (reference "R6") (unit 1) (value "470") (footprint "ukmarsbot:R_Axial_DIN0207_L6.3mm_D2.5mm_P7.62mm_BIGPAD")
     )
     (path "/1f6d8026-88d7-4db1-9273-bc8270850418"
-      (reference "R7") (unit 1) (value "15k") (footprint "ukmarsbot:R_Axial_DIN0207_L6.3mm_D2.5mm_P7.62mm_Horizontal")
+      (reference "R7") (unit 1) (value "15k") (footprint "ukmarsbot:R_Axial_DIN0207_L6.3mm_D2.5mm_P7.62mm_BIGPAD")
     )
     (path "/62359ea0-0ee0-4e05-b793-eb25752a39f7"
-      (reference "R8") (unit 1) (value "15k") (footprint "ukmarsbot:R_Axial_DIN0207_L6.3mm_D2.5mm_P7.62mm_Horizontal")
+      (reference "R8") (unit 1) (value "15k") (footprint "ukmarsbot:R_Axial_DIN0207_L6.3mm_D2.5mm_P7.62mm_BIGPAD")
     )
     (path "/10dfea55-4def-445e-b233-52b194366676"
-      (reference "R10") (unit 1) (value "10k") (footprint "ukmarsbot:R_Axial_DIN0207_L6.3mm_D2.5mm_P7.62mm_Horizontal")
+      (reference "R10") (unit 1) (value "10k") (footprint "ukmarsbot:R_Axial_DIN0207_L6.3mm_D2.5mm_P7.62mm_BIGPAD")
     )
     (path "/2c389bd4-3c3f-4b2d-a7ca-5c224974629f"
-      (reference "R11") (unit 1) (value "4k7") (footprint "ukmarsbot:R_Axial_DIN0207_L6.3mm_D2.5mm_P7.62mm_Horizontal")
+      (reference "R11") (unit 1) (value "4k7") (footprint "ukmarsbot:R_Axial_DIN0207_L6.3mm_D2.5mm_P7.62mm_BIGPAD")
     )
     (path "/e3713f85-2a22-40fc-8498-9a1d5ba496c5"

Commit message: Update V1.3 mainboard BOM
Parts:
- C2, C3: Note (none) -> Maximum height is 10mm
- D1: Note (none) -> > 2A rectifier. Shottky is good
- H1, H2, H3, H4, H5, H6: Note (none) -> Check finished size is M3 (3.2mm)
- J1: Note (none) -> 14 pin header, 0.1", male
- J2, J3: Note (none) -> 6 pin header, 0.1", male
- J4: Note (none) -> 0.1" pitch, polarised, any type
- J5: Note (none) -> 4 pin, 0.1", male
- M1, M2: Note (none) -> commercial mounts need bushing for screws
- R1, R10, R11, R2, R3, R4, R5, R6, R7, R8: Note (none) -> any type, but small, 0.2" span
- S1: Note (none) -> Toggle or slide, 0.1" pitch pins
- S2: Note (none) -> Check orientation
- S3: Note (none) -> Check orientation. On is towards front
- U2: Note (none) -> Check orientation. Only Sparkfun layout supported
Changed lines of the file:
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@@
+      (effects (font (size 1.27 1.27)) hide)
+    )
+    (property "Note" "any type, but small, 0.2\" span" (id 4) (at 46.99 31.75 0)
       (effects (font (size 1.27 1.27)) hide)
     )
@@
     )
     (property "Datasheet" "~" (id 3) (at 165.1 148.59 0)
+      (effects (font (size 1.27 1.27)) hide)
+    )
+    (property "Note" "any type, but small, 0.2\" span" (id 4) (at 165.1 148.59 0)
       (effects (font (size 1.27 1.27)) hide)
     )
@@
     )
     (property "Datasheet" "~" (id 3) (at 254 48.26 0)
+      (effects (font (size 1.27 1.27)) hide)
+    )
+    (property "Note" "any type, but small, 0.2\" span" (id 4) (at 254 48.26 0)
       (effects (font (size 1.27 1.27)) hide)
     )
@@
       (effects (font (size 1.27 1.27)) hide)
     )
+    (property "Note" "any type, but small, 0.2\" span" (id 4) (at 54.61 19.05 0)
+      (effects (font (size 1.27 1.27)) hide)
+    )
     (pin "1")
     (pin "2")
@@
       (effects (font (size 1.27 1.27)) hide)
     )
+    (property "Note" "Check orientation. On is towards front" (id 4) (at 134.62 140.97 0)
+      (effects (font (size 1.27 1.27)) hide)
+    )
     (pin "1")
     (pin "8")
@@
       (effects (font (size 1.27 1.27)) hide)
     )
+    (property "Note" "6 pin header, 0.1\", male" (id 4) (at 30.48 133.35 0)
+      (effects (font (size 1.27 1.27)) hide)
+    )
     (pin "1")
     (pin "2")
@@
       (effects (font (size 1.27 1.27)) hide)
     )
+    (property "Note" "any type, but small, 0.2\" span" (id 4) (at 172.72 156.21 0)
+      (effects (font (size 1.27 1.27)) hide)
+    )
     (pin "1")
     (pin "2")
@@
     )
     (property "Datasheet" "~" (id 3) (at 119.38 148.59 0)
+      (effects (font (size 1.27 1.27)) hide)
+    )
+    (property "Note" "any type, but small, 0.2\" span" (id 4) (at 119.38 148.59 0)
       (effects (font (size 1.27 1.27)) hide)
     )
@@
     )
     (property "Datasheet" "" (id 3) (at 20.32 24.13 0)
+      (effects (font (size 1.27 1.27)) hide)
+    )
+    (property "Note" "4 pin, 0.1\", male" (id 4) (at 20.32 24.13 0)
       (effects (font (size 1.27 1.27)) hide)
     )
@@
       (effects (font (size 1.27 1.27)) hide)
     )
+    (property "Note" "any type, but small, 0.2\" span" (id 4) (at 104.14 133.35 0)
+      (effects (font (size 1.27 1.27)) hide)
+    )
     (pin "1")
     (pin "2")
@@
     )
     (property "Datasheet" "~" (id 3) (at 254 66.04 0)
+      (effects (font (size 1.27 1.27)) hide)
+    )
+    (property "Note" "any type, but small, 0.2\" span" (id 4) (at 254 66.04 0)
       (effects (font (size 1.27 1.27)) hide)
     )
@@
       (effects (font (size 1.27 1.27)) hide)
     )
+    (property "Note" "Check finished size is M3 (3.2mm)" (id 4) (at 99.06 173.99 0)
+      (effects (font (size 1.27 1.27)) hide)
+    )
   )
   (symbol (lib_id "power:GND") (at 77.47 88.9 0) (unit 1)
@@
     )
     (property "Datasheet" "~" (id 3) (at 200.66 36.83 0)
+      (effects (font (size 1.27 1.27)) hide)
+    )
+    (property "Note" "0.1\" pitch, polarised, any type" (id 4) (at 200.66 36.83 0)
       (effects (font (size 1.27 1.27)) hide)
     )
@@
       (effects (font (size 1.27 1.27)) (justify left bottom) hide)
     )
-    (property "Datasheet" "" (id 3) (at 153.67 88.9 0)
+    (property "Datasheet" "https://cdn.shopify.com/s/files/1/0174/1800/files/TB6612FNG_3e2152f9-ac47-436b-bb2d-0abf1ce342e0.pdf?15448876658223299941" (id 3) (at 153.67 88.9 0)
       (effects (font (size 1.27 1.27)) (justify left bottom) hide)
     )
@@
     (property "PARTREV" "11-13-17" (id 6) (at 153.67 88.9 0)
       (effects (font (size 1.27 1.27)) (justify left bottom) hide)
+    )
+    (property "Note" "Check orientation. Only Sparkfun layout supported" (id 7) (at 153.67 88.9 0)
+      (effects (font (size 1.27 1.27)) hide)
     )
     (pin "1")
@@
       (effects (font (size 1.27 1.27)) hide)
     )
+    (property "Note" "Maximum height is 10mm" (id 4) (at 96.52 81.28 0)
+      (effects (font (size 1.27 1.27)) hide)
+    )
     (pin "1")
     (pin "2")
@@
     )
     (property "Datasheet" "~" (id 3) (at 135.89 148.59 0)
+      (effects (font (size 1.27 1.27)) hide)
+    )
+    (property "Note" "any type, but small, 0.2\" span" (id 4) (at 135.89 148.59 0)
       (effects (font (size 1.27 1.27)) hide)
     )
@@
       (effects (font (size 1.27 1.27)) hide)
     )
+    (property "Note" "> 2A rectifier. Shottky is good" (id 4) (at 247.65 36.83 0)
+      (effects (font (size 1.27 1.27)) hide)
+    )
     (pin "1")
     (pin "2")
@@
     )
     (property "Datasheet" "~" (id 3) (at 99.06 181.61 0)
+      (effects (font (size 1.27 1.27)) hide)
+    )
+    (property "Note" "Check finished size is M3 (3.2mm)" (id 4) (at 99.06 181.61 0)
       (effects (font (size 1.27 1.27)) hide)
     )
@@
     )
     (property "Datasheet" "" (id 3) (at 119.38 140.97 0)
+      (effects (font (size 1.27 1.27)) hide)
+    )
+    (property "Note" "Check orientation. On is towards front" (id 4) (at 119.38 140.97 0)
       (effects (font (size 1.27 1.27)) hide)
     )
@@
       (effects (font (size 1.27 1.27)) hide)
     )
+    (property "Note" "Check orientation. On is towards front" (id 4) (at 149.86 140.97 0)
+      (effects (font (size 1.27 1.27)) hide)
+    )
     (pin "1")
     (pin "8")
@@
       (effects (font (size 1.27 1.27)) hide)
     )
+    (property "Note" "6 pin header, 0.1\", male" (id 4) (at 30.48 168.91 0)
+      (effects (font (size 1.27 1.27)) hide)
+    )
     (pin "1")
     (pin "2")
@@
       (effects (font (size 1.27 1.27)) hide)
     )
+    (property "Note" "Maximum height is 10mm" (id 4) (at 77.47 81.28 0)
+      (effects (font (size 1.27 1.27)) hide)
+    )
     (pin "1")
     (pin "2")
@@
       (effects (font (size 1.27 1.27)) hide)
     )
+    (property "Note" "Check finished size is M3 (3.2mm)" (id 4) (at 118.11 181.61 0)
+      (effects (font (size 1.27 1.27)) hide)
+    )
   )
   (symbol (lib_id "Mechanical:MountingHole") (at 78.74 173.99 0) (unit 1)
@@
       (effects (font (size 1.27 1.27)) hide)
     )
+    (property "Note" "Check finished size is M3 (3.2mm)" (id 4) (at 78.74 173.99 0)
+      (effects (font (size 1.27 1.27)) hide)
+    )
   )
   (symbol (lib_id "ukmarsbot:GEARMOTOR") (at 106.68 101.6 0) (unit 1)
@@
     )
     (property "Datasheet" "~" (id 3) (at 106.68 102.616 0)
+      (effects (font (size 1.27 1.27)) hide)
+    )
+    (property "Note" "commercial mounts need bushing for screws" (id 4) (at 106.68 101.6 0)
       (effects (font (size 1.27 1.27)) hide)
     )
@@
       (effects (font (size 1.27 1.27)) hide)
     )
+    (property "Note" "Check orientation" (id 4) (at 93.98 133.35 0)
+      (effects (font (size 1.27 1.27)) hide)
+    )
     (pin "1")
     (pin "2")
@@
     )
     (property "Datasheet" "~" (id 3) (at 151.13 148.59 0)
+      (effects (font (size 1.27 1.27)) hide)
+    )
+    (property "Note" "any type, but small, 0.2\" span" (id 4) (at 151.13 148.59 0)
       (effects (font (size 1.27 1.27)) hide)
     )
@@
       (effects (font (size 1.27 1.27)) hide)
     )
+    (property "Note" "Check finished size is M3 (3.2mm)" (id 4) (at 118.11 173.99 0)
+      (effects (font (size 1.27 1.27)) hide)
+    )
   )
   (symbol (lib_id "ukmarsbot:SWITCH-SPDT-PTH-11.6X4.0MM") (at 227.33 34.29 0) (unit 1)
@@
       (effects (font (size 1.27 1.27)) hide)
     )
+    (property "Note" "Toggle or slide, 0.1\" pitch pins" (id 4) (at 227.33 34.29 0)
+      (effects (font (size 1.27 1.27)) hide)
+    )
     (pin "1")
     (pin "2")
@@
     )
     (property "Datasheet" "" (id 3) (at 165.1 140.97 0)
+      (effects (font (size 1.27 1.27)) hide)
+    )
+    (property "Note" "Check orientation. On is towards front" (id 4) (at 165.1 140.97 0)
       (effects (font (size 1.27 1.27)) hide)
     )
@@
       (effects (font (size 1.27 1.27)) hide)
     )
+    (property "Note" "14 pin header, 0.1\", male" (id 4) (at 25.4 80.01 0)
+      (effects (font (size 1.27 1.27)) hide)
+    )
     (pin "1")
     (pin "10")
@@
       (effects (font (size 1.27 1.27)) hide)
     )
+    (property "Note" "commercial mounts need bushing for screws" (id 4) (at 78.74 101.6 0)
+      (effects (font (size 1.27 1.27)) hide)
+    )
   )
   (symbol (lib_id "Mechanical:MountingHole") (at 78.74 181.61 0) (unit 1)
@@
       (effects (font (size 1.27 1.27)) hide)
     )
+    (property "Note" "Check finished size is M3 (3.2mm)" (id 4) (at 78.74 181.61 0)
+      (effects (font (size 1.27 1.27)) hide)
+    )

Commit message: updare mounting holes V1.3 mainboard
update V1.3 mainboard mounting holes
Parts:
- H1, H2, H3, H4, H5, H6: footprint MountingHole:MountingHole_3.2mm_M3 -> ukmarsbot:MountingHole_3.2mm_M3_clearance
Changed lines of the file:
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@@
       (effects (font (size 1.27 1.27)) (justify left))
     )
-    (property "Footprint" "MountingHole:MountingHole_3.2mm_M3" (id 2) (at 99.06 173.99 0)
+    (property "Footprint" "ukmarsbot:MountingHole_3.2mm_M3_clearance" (id 2) (at 99.06 173.99 0)
       (effects (font (size 1.27 1.27)) hide)
     )
@@
       (effects (font (size 1.27 1.27)) (justify left))
     )
-    (property "Footprint" "MountingHole:MountingHole_3.2mm_M3" (id 2) (at 99.06 181.61 0)
+    (property "Footprint" "ukmarsbot:MountingHole_3.2mm_M3_clearance" (id 2) (at 99.06 181.61 0)
       (effects (font (size 1.27 1.27)) hide)
     )
@@
       (effects (font (size 1.27 1.27)) (justify left))
     )
-    (property "Footprint" "MountingHole:MountingHole_3.2mm_M3" (id 2) (at 118.11 181.61 0)
+    (property "Footprint" "ukmarsbot:MountingHole_3.2mm_M3_clearance" (id 2) (at 118.11 181.61 0)
       (effects (font (size 1.27 1.27)) hide)
     )
@@
       (effects (font (size 1.27 1.27)) (justify left))
     )
-    (property "Footprint" "MountingHole:MountingHole_3.2mm_M3" (id 2) (at 78.74 173.99 0)
+    (property "Footprint" "ukmarsbot:MountingHole_3.2mm_M3_clearance" (id 2) (at 78.74 173.99 0)
       (effects (font (size 1.27 1.27)) hide)
     )
@@
       (effects (font (size 1.27 1.27)) (justify left))
     )
-    (property "Footprint" "MountingHole:MountingHole_3.2mm_M3" (id 2) (at 118.11 173.99 0)
+    (property "Footprint" "ukmarsbot:MountingHole_3.2mm_M3_clearance" (id 2) (at 118.11 173.99 0)
       (effects (font (size 1.27 1.27)) hide)
     )
@@
       (effects (font (size 1.27 1.27)) (justify left))
     )
-    (property "Footprint" "MountingHole:MountingHole_3.2mm_M3" (id 2) (at 78.74 181.61 0)
+    (property "Footprint" "ukmarsbot:MountingHole_3.2mm_M3_clearance" (id 2) (at 78.74 181.61 0)
       (effects (font (size 1.27 1.27)) hide)
     )
@@
     )
     (path "/cc0bfa2d-8e97-4239-8fea-fc713b9750e0"
-      (reference "H1") (unit 1) (value "MountingHole") (footprint "MountingHole:MountingHole_3.2mm_M3")
+      (reference "H1") (unit 1) (value "MountingHole") (footprint "ukmarsbot:MountingHole_3.2mm_M3_clearance")
     )
     (path "/fb4e89f0-1d7c-437a-aed8-64f86da5d5be"
-      (reference "H2") (unit 1) (value "MountingHole") (footprint "MountingHole:MountingHole_3.2mm_M3")
+      (reference "H2") (unit 1) (value "MountingHole") (footprint "ukmarsbot:MountingHole_3.2mm_M3_clearance")
     )
     (path "/6f1b992c-589d-4950-aca9-a939f6e742a4"
-      (reference "H3") (unit 1) (value "MountingHole") (footprint "MountingHole:MountingHole_3.2mm_M3")
+      (reference "H3") (unit 1) (value "MountingHole") (footprint "ukmarsbot:MountingHole_3.2mm_M3_clearance")
     )
     (path "/865301db-2325-4385-92b8-a436a149e286"
-      (reference "H4") (unit 1) (value "MountingHole") (footprint "MountingHole:MountingHole_3.2mm_M3")
+      (reference "H4") (unit 1) (value "MountingHole") (footprint "ukmarsbot:MountingHole_3.2mm_M3_clearance")
     )
     (path "/e2d7f4f3-be03-49a8-84ed-d4db5647a76e"
-      (reference "H5") (unit 1) (value "MountingHole") (footprint "MountingHole:MountingHole_3.2mm_M3")
+      (reference "H5") (unit 1) (value "MountingHole") (footprint "ukmarsbot:MountingHole_3.2mm_M3_clearance")
     )
     (path "/c4046656-9af6-49f9-ad02-d1a389c36423"
-      (reference "H6") (unit 1) (value "MountingHole") (footprint "MountingHole:MountingHole_3.2mm_M3")
+      (reference "H6") (unit 1) (value "MountingHole") (footprint "ukmarsbot:MountingHole_3.2mm_M3_clearance")
     )
     (path "/6ce108c9-a3af-4009-9386-a52e62b85247"

Commit message: update V1.3 mainboard switches
Parts:
- S1: footprint ukmarsbot:SW_1101M2S3CQE2 -> ukmarsbot:SW_MINI_SPDT_TOGGLE_DAILYWELL_FS1S102M2QES; Note Toggle or slide, 0.1" pitch pins -> Toggle or slide, 0.1" pitch pins, EG Salecom TS-4-TE1CR-E-H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; Vendor (none) -> https://www.rapidonline.com/salecom-ts-4-te1cr-e-h-z03-spdt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
Changed lines of the file:
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@@
       (effects (font (size 1.778 1.778)) (justify top))
     )
-    (property "Footprint" "ukmarsbot:SW_1101M2S3CQE2" (id 2) (at 227.33 34.29 0)
-      (effects (font (size 1.27 1.27)) hide)
-    )
-    (property "Datasheet" "" (id 3) (at 227.33 34.29 0)
-      (effects (font (size 1.27 1.27)) hide)
-    )
-    (property "Note" "Toggle or slide, 0.1\" pitch pins" (id 4) (at 227.33 34.29 0)
+    (property "Footprint" "ukmarsbot:SW_MINI_SPDT_TOGGLE_DAILYWELL_FS1S102M2QES" (id 2) (at 227.33 34.29 0)
+      (effects (font (size 1.27 1.27)) hide)
+    )
+    (property "Datasheet" "https://static.rapidonline.com/pdf/560602t_v1.pdf" (id 3) (at 227.33 34.29 0)
+      (effects (font (size 1.27 1.27)) hide)
+    )
+    (property "Note" "Toggle or slide, 0.1\" pitch pins, EG Salecom TS-4-TE1CR-E-H-Z03" (id 4) (at 227.33 34.29 0)
+      (effects (font (size 1.27 1.27)) hide)
+    )
+    (property "Vendor" "https://www.rapidonline.com/salecom-ts-4-te1cr-e-h-z03-spdt-sub-min-vertical-pcb-toggle-switch-75-0238" (id 5) (at 227.33 34.29 0)
       (effects (font (size 1.27 1.27)) hide)
     )
@@
     )
     (path "/e3713f85-2a22-40fc-8498-9a1d5ba496c5"
-      (reference "S1") (unit 1) (value "sub-miniature, SPDT") (footprint "ukmarsbot:SW_1101M2S3CQE2")
+      (reference "S1") (unit 1) (value "sub-miniature, SPDT") (footprint "ukmarsbot:SW_MINI_SPDT_TOGGLE_DAILYWELL_FS1S102M2QES")
     )
     (path "/d0feb225-71a8-4533-9b0a-f0eabf97a0e5"
