File: ecad/kicad/wall-sensor-advanced/ukmarsbot-wall-sensor-advanced.kicad_sch (KiCad schematic)
At the start: 29 parts, among them J1 Conn_01x14, Q1 TEFT4300, Q2 TEFT4300, Q3 TEFT4300, Q4 TEFT4300, Q5 BC337, Q6 BC337

Commit message: second draft wall sensor advanced
Parts:
- added C2: 330uF, 16V, Capacitor_THT:CP_Radial_D7.5mm_P2.50mm, symbol Device:C_Polarized
Connections:
- net +5V: now also C2.1
- net GND: now also C2.2
- net DIA_COMMON: now reaches D2.1 (K), D3.1 (K), Q6.1 (C)
- net FWD_COMMON: now reaches D1.1 (K), D4.1 (K), Q5.1 (C)
Changed lines of the file:
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@@
+    (stroke (width 0) (type default) (color 0 0 0 0))
+  )
+  (wire (pts (xy 96.52 167.64) (xy 96.52 176.53))
     (stroke (width 0) (type default) (color 0 0 0 0))
   )
@@
   )
   (wire (pts (xy 148.59 57.15) (xy 148.59 58.42))
+    (stroke (width 0) (type default) (color 0 0 0 0))
+  )
+  (wire (pts (xy 96.52 149.86) (xy 96.52 160.02))
     (stroke (width 0) (type default) (color 0 0 0 0))
   )
@@
   (label "D11_FRONT" (at 120.65 134.62 0)
     (effects (font (size 1.0922 1.0922)) (justify left bottom))
+  )
+  (label "DIA_COMMON" (at 198.12 129.54 0)
+    (effects (font (size 1.27 1.27)) (justify left bottom))
+  )
+  (label "FWD_COMMON" (at 149.86 129.54 0)
+    (effects (font (size 1.27 1.27)) (justify left bottom))
   )
   (global_label "A2_LD" (shape input) (at 35.56 95.25 0) (fields_autoplaced)
@@
     (pin "2")
   )
+  (symbol (lib_id "power:+5V") (at 96.52 149.86 0) (unit 1)
+    (in_bom yes) (on_board yes)
+    (property "Reference" "#PWR0101" (id 0) (at 96.52 153.67 0)
+      (effects (font (size 1.27 1.27)) hide)
+    )
+    (property "Value" "+5V" (id 1) (at 96.901 145.4658 0))
+    (property "Footprint" "" (id 2) (at 96.52 149.86 0)
+      (effects (font (size 1.27 1.27)) hide)
+    )
+    (property "Datasheet" "" (id 3) (at 96.52 149.86 0)
+      (effects (font (size 1.27 1.27)) hide)
+    )
+    (pin "1")
+  )
   (symbol (lib_id "Device:R") (at 181.61 134.62 90) (unit 1)
     (in_bom yes) (on_board yes)
@@
     (pin "1")
   )
+  (symbol (lib_id "Device:C_Polarized") (at 96.52 163.83 0) (unit 1)
+    (in_bom yes) (on_board yes)
+    (property "Reference" "C2" (id 0) (at 99.5172 162.6616 0)
+      (effects (font (size 1.27 1.27)) (justify left))
+    )
+    (property "Value" "330uF, 16V" (id 1) (at 99.5172 164.973 0)
+      (effects (font (size 1.27 1.27)) (justify left))
+    )
+    (property "Footprint" "Capacitor_THT:CP_Radial_D7.5mm_P2.50mm" (id 2) (at 97.4852 167.64 0)
+      (effects (font (size 1.27 1.27)) hide)
+    )
+    (property "Datasheet" "~" (id 3) (at 96.52 163.83 0)
+      (effects (font (size 1.27 1.27)) hide)
+    )
+    (pin "1")
+    (pin "2")
+  )
+  (symbol (lib_id "power:GND") (at 96.52 176.53 0) (unit 1)
+    (in_bom yes) (on_board yes)
+    (property "Reference" "#PWR0102" (id 0) (at 96.52 182.88 0)
+      (effects (font (size 1.27 1.27)) hide)
+    )
+    (property "Value" "GND" (id 1) (at 96.647 180.9242 0))
+    (property "Footprint" "" (id 2) (at 96.52 176.53 0)
+      (effects (font (size 1.27 1.27)) hide)
+    )
+    (property "Datasheet" "" (id 3) (at 96.52 176.53 0)
+      (effects (font (size 1.27 1.27)) hide)
+    )
+    (pin "1")
+  )
   (sheet_instances
     (path "/" (page "1"))
@@
       (reference "#PWR015") (unit 1) (value "GND") (footprint "")
     )
+    (path "/5200118b-6a39-4f0f-9a39-9d6a4cf0be3a"
+      (reference "#PWR0101") (unit 1) (value "+5V") (footprint "")
+    )
+    (path "/bba69b9e-c692-4e50-b429-c633985bea15"
+      (reference "#PWR0102") (unit 1) (value "GND") (footprint "")
+    )
     (path "/00000000-0000-0000-0000-000060b75527"
       (reference "C1") (unit 1) (value "330uF, 16V") (footprint "Capacitor_THT:CP_Radial_D7.5mm_P2.50mm")
     )
+    (path "/a785db99-bc5e-4380-a605-b134409d112a"
+      (reference "C2") (unit 1) (value "330uF, 16V") (footprint "Capacitor_THT:CP_Radial_D7.5mm_P2.50mm")
+    )
     (path "/00000000-0000-0000-0000-000060ae73d0"

Commit message: Update Advanced Wall Sensor
Parts:
- C1, C2: footprint Capacitor_THT:CP_Radial_D7.5mm_P2.50mm -> Capacitor_THT:CP_Radial_D10.0mm_P2.50mm
- D1, D2, D3, D4: footprint LED_THT:LED_D5.0mm_Horizontal_O3.81mm_Z3.0mm -> ukmarsbot:LED_D5.0mm_Horizontal_O6.35mm_Z3.0mm
- J1: footprint Connector_PinSocket_2.54mm:PinSocket_1x14_P2.54mm_Vertical -> ukmarsbot:PinHeader_1x14_P2.54mm_Vertical_Longpads
- Q1, Q2, Q3, Q4: footprint LED_THT:LED_D5.0mm_Horizontal_O1.27mm_Z3.0mm_IRGrey -> ukmarsbot:LED_D5.0mm_Horizontal_O1.27mm_Z3.0mm_IRGrey
- R5, R6, R7, R8: value 2k7 -> 1k8
Other:
- note added: "Advanced Wall Sensor for Maze Solvers"
- note added: "Detector Phototransistors"
- note added: "General Purpose Indicator"
- note added: "Power Supply and smoothing"
- note added: "Resistors R1, R2, R3 and R4 will be adjusted on test to suit the emitters in use. Current for the emitters is drawn from the capacitor C1. LEDs D1, D2, D3 and D4 may be high intensity red, blue or IR emitters. Whatever is chosen, take care that the detectors, Q3-6 are spectrally matched. An alternative to the SFH4550 IR emitters might be super bright red LEDs such as the TLCR5800 paired with BPW9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"
- note added: "Sensor Connector"
- note added: "Smoothing capacitors should be 16V types and no more than 10mm diameter. Put in the largest value you can find. R11 may need to be adjusted to ensure that charge is not lost from C1 when sensors are operating. Note that R11 sets the maximum current through the emitters if they are accidentally left on."
- note added: "Spacers of 11.25mm are needed between the sensor board and the mainboard to match the typical height of the combined pin header and socket of the sensor connector"
- note added: "The sensor connector would be a 14 pin SIL socket to push directly onto the sensor header on the mainboard"
- note removed: "Resistors R1, R3, R4 and R6 will be adjusted on test to suit the emitters in use. Current for the emitters is drawn from the capacitor C1, LEDs D1, D2, D3 and D4 may be high intensity red, blue or IR emitters. Whatever is chosen, take care that the detectors, Q3-6 are spectrally matched. NOTE that high-power IR emitters such as the SFH4550 may present a possible eye safety hazard and should not b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"
- moved on the sheet: C1, C2, D5, R11, R12

Commit message: correct net name error on adv wall sensor
Connections:
- net A0_LF renamed A0_RF
Changed lines of the file:
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@@
     )
   )
-  (global_label "A0_LF" (shape input) (at 195.58 57.15 0) (fields_autoplaced)
+  (global_label "A0_RF" (shape input) (at 195.58 57.15 0) (fields_autoplaced)
     (effects (font (size 1.27 1.27)) (justify left))
-    (property "Intersheet References" "${INTERSHEET_REFS}" (id 0) (at 24.13 -35.56 0)
-      (effects (font (size 1.27 1.27)) hide)
+    (property "Intersheet References" "${INTERSHEET_REFS}" (id 0) (at 203.5285 57.0706 0)
+      (effects (font (size 1.27 1.27)) (justify left) hide)
     )
   )
@@
     )
   )
-  (global_label "A0_LF" (shape input) (at 35.56 100.33 0) (fields_autoplaced)
+  (global_label "A0_RF" (shape input) (at 35.56 100.33 0) (fields_autoplaced)
     (effects (font (size 1.0922 1.0922)) (justify left))
-    (property "Intersheet References" "${INTERSHEET_REFS}" (id 0) (at -27.94 -45.72 0)
-      (effects (font (size 1.27 1.27)) hide)
+    (property "Intersheet References" "${INTERSHEET_REFS}" (id 0) (at 42.3956 100.2618 0)
+      (effects (font (size 1.0922 1.0922)) (justify left) hide)
     )
   )

Commit message: use bigpad resistors on adv wall sensor
Parts:
- R1, R10, R11, R12, R13, R14, R2, R3, R4, R5, R6, R7, R8, R9: footprint ukmarsbot:R_Axial_DIN0207_L6.3mm_D2.5mm_P7.62mm_Horizontal -> ukmarsbot:R_Axial_DIN0207_L6.3mm_D2.5mm_P7.62mm_BIGPAD
Changed lines of the file:
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@@
       (effects (font (size 1.27 1.27)) (justify left))
     )
-    (property "Footprint" "ukmarsbot:R_Axial_DIN0207_L6.3mm_D2.5mm_P7.62mm_Horizontal" (id 2) (at 189.992 62.23 90)
+    (property "Footprint" "ukmarsbot:R_Axial_DIN0207_L6.3mm_D2.5mm_P7.62mm_BIGPAD" (id 2) (at 189.992 62.23 90)
       (effects (font (size 1.27 1.27)) hide)
     )
@@
       (effects (font (size 1.27 1.27)) (justify left))
     )
-    (property "Footprint" "ukmarsbot:R_Axial_DIN0207_L6.3mm_D2.5mm_P7.62mm_Horizontal" (id 2) (at 146.812 62.23 90)
+    (property "Footprint" "ukmarsbot:R_Axial_DIN0207_L6.3mm_D2.5mm_P7.62mm_BIGPAD" (id 2) (at 146.812 62.23 90)
       (effects (font (size 1.27 1.27)) hide)
     )
@@
       (effects (font (size 1.27 1.27)) (justify left))
     )
-    (property "Footprint" "ukmarsbot:R_Axial_DIN0207_L6.3mm_D2.5mm_P7.62mm_Horizontal" (id 2) (at 168.402 62.23 90)
+    (property "Footprint" "ukmarsbot:R_Axial_DIN0207_L6.3mm_D2.5mm_P7.62mm_BIGPAD" (id 2) (at 168.402 62.23 90)
       (effects (font (size 1.27 1.27)) hide)
     )
@@
       (effects (font (size 1.27 1.27)) (justify left))
     )
-    (property "Footprint" "ukmarsbot:R_Axial_DIN0207_L6.3mm_D2.5mm_P7.62mm_Horizontal" (id 2) (at 185.928 111.76 90)
+    (property "Footprint" "ukmarsbot:R_Axial_DIN0207_L6.3mm_D2.5mm_P7.62mm_BIGPAD" (id 2) (at 185.928 111.76 90)
       (effects (font (size 1.27 1.27)) hide)
     )
@@
       (effects (font (size 1.27 1.27)) (justify left))
     )
-    (property "Footprint" "ukmarsbot:R_Axial_DIN0207_L6.3mm_D2.5mm_P7.62mm_Horizontal" (id 2) (at 151.638 111.76 90)
+    (property "Footprint" "ukmarsbot:R_Axial_DIN0207_L6.3mm_D2.5mm_P7.62mm_BIGPAD" (id 2) (at 151.638 111.76 90)
       (effects (font (size 1.27 1.27)) hide)
     )
@@
       (effects (font (size 1.27 1.27)) (justify right))
     )
-    (property "Footprint" "ukmarsbot:R_Axial_DIN0207_L6.3mm_D2.5mm_P7.62mm_Horizontal" (id 2) (at 137.922 139.7 90)
+    (property "Footprint" "ukmarsbot:R_Axial_DIN0207_L6.3mm_D2.5mm_P7.62mm_BIGPAD" (id 2) (at 137.922 139.7 90)
       (effects (font (size 1.27 1.27)) hide)
     )
@@
       (effects (font (size 1.27 1.27)) (justify left))
     )
-    (property "Footprint" "ukmarsbot:R_Axial_DIN0207_L6.3mm_D2.5mm_P7.62mm_Horizontal" (id 2) (at 137.668 111.76 90)
+    (property "Footprint" "ukmarsbot:R_Axial_DIN0207_L6.3mm_D2.5mm_P7.62mm_BIGPAD" (id 2) (at 137.668 111.76 90)
       (effects (font (size 1.27 1.27)) hide)
     )
@@
       (effects (font (size 1.27 1.27)) (justify left))
     )
-    (property "Footprint" "ukmarsbot:R_Axial_DIN0207_L6.3mm_D2.5mm_P7.62mm_Horizontal" (id 2) (at 199.898 111.76 90)
+    (property "Footprint" "ukmarsbot:R_Axial_DIN0207_L6.3mm_D2.5mm_P7.62mm_BIGPAD" (id 2) (at 199.898 111.76 90)
       (effects (font (size 1.27 1.27)) hide)
     )
@@
       (effects (font (size 1.27 1.27)) (justify left))
     )
-    (property "Footprint" "ukmarsbot:R_Axial_DIN0207_L6.3mm_D2.5mm_P7.62mm_Horizontal" (id 2) (at 125.222 62.23 90)
+    (property "Footprint" "ukmarsbot:R_Axial_DIN0207_L6.3mm_D2.5mm_P7.62mm_BIGPAD" (id 2) (at 125.222 62.23 90)
       (effects (font (size 1.27 1.27)) hide)
     )
@@
       (effects (font (size 1.27 1.27)) (justify right))
     )
-    (property "Footprint" "ukmarsbot:R_Axial_DIN0207_L6.3mm_D2.5mm_P7.62mm_Horizontal" (id 2) (at 186.182 139.7 90)
+    (property "Footprint" "ukmarsbot:R_Axial_DIN0207_L6.3mm_D2.5mm_P7.62mm_BIGPAD" (id 2) (at 186.182 139.7 90)
       (effects (font (size 1.27 1.27)) hide)
     )
@@
       (effects (font (size 1.27 1.27)) (justify right))
     )
-    (property "Footprint" "ukmarsbot:R_Axial_DIN0207_L6.3mm_D2.5mm_P7.62mm_Horizontal" (id 2) (at 43.688 151.13 90)
+    (property "Footprint" "ukmarsbot:R_Axial_DIN0207_L6.3mm_D2.5mm_P7.62mm_BIGPAD" (id 2) (at 43.688 151.13 90)
       (effects (font (size 1.27 1.27)) hide)
     )
@@
       (effects (font (size 1.27 1.27)) (justify right))
     )
-    (property "Footprint" "ukmarsbot:R_Axial_DIN0207_L6.3mm_D2.5mm_P7.62mm_Horizontal" (id 2) (at 67.818 148.59 90)
+    (property "Footprint" "ukmarsbot:R_Axial_DIN0207_L6.3mm_D2.5mm_P7.62mm_BIGPAD" (id 2) (at 67.818 148.59 90)
       (effects (font (size 1.27 1.27)) hide)
     )
@@
       (effects (font (size 1.27 1.27)) (justify left))
     )
-    (property "Footprint" "ukmarsbot:R_Axial_DIN0207_L6.3mm_D2.5mm_P7.62mm_Horizontal" (id 2) (at 133.35 136.398 90)
+    (property "Footprint" "ukmarsbot:R_Axial_DIN0207_L6.3mm_D2.5mm_P7.62mm_BIGPAD" (id 2) (at 133.35 136.398 90)
       (effects (font (size 1.27 1.27)) hide)
     )
@@
       (effects (font (size 1.27 1.27)) (justify left))
     )
-    (property "Footprint" "ukmarsbot:R_Axial_DIN0207_L6.3mm_D2.5mm_P7.62mm_Horizontal" (id 2) (at 181.61 136.398 90)
+    (property "Footprint" "ukmarsbot:R_Axial_DIN0207_L6.3mm_D2.5mm_P7.62mm_BIGPAD" (id 2) (at 181.61 136.398 90)
       (effects (font (size 1.27 1.27)) hide)
     )
@@
     )
     (path "/00000000-0000-0000-0000-000060ae73d6"
-      (reference "R1") (unit 1) (value "10R") (footprint "ukmarsbot:R_Axial_DIN0207_L6.3mm_D2.5mm_P7.62mm_Horizontal")
+      (reference "R1") (unit 1) (value "10R") (footprint "ukmarsbot:R_Axial_DIN0207_L6.3mm_D2.5mm_P7.62mm_BIGPAD")
     )
     (path "/00000000-0000-0000-0000-000060adf19e"
-      (reference "R2") (unit 1) (value "10R") (footprint "ukmarsbot:R_Axial_DIN0207_L6.3mm_D2.5mm_P7.62mm_Horizontal")
+      (reference "R2") (unit 1) (value "10R") (footprint "ukmarsbot:R_Axial_DIN0207_L6.3mm_D2.5mm_P7.62mm_BIGPAD")
     )
     (path "/00000000-0000-0000-0000-000060aeae98"
-      (reference "R3") (unit 1) (value "10R") (footprint "ukmarsbot:R_Axial_DIN0207_L6.3mm_D2.5mm_P7.62mm_Horizontal")
+      (reference "R3") (unit 1) (value "10R") (footprint "ukmarsbot:R_Axial_DIN0207_L6.3mm_D2.5mm_P7.62mm_BIGPAD")
     )
     (path "/00000000-0000-0000-0000-000060ae7394"
-      (reference "R4") (unit 1) (value "10R") (footprint "ukmarsbot:R_Axial_DIN0207_L6.3mm_D2.5mm_P7.62mm_Horizontal")
+      (reference "R4") (unit 1) (value "10R") (footprint "ukmarsbot:R_Axial_DIN0207_L6.3mm_D2.5mm_P7.62mm_BIGPAD")
     )
     (path "/00000000-0000-0000-0000-000060aec69c"
-      (reference "R5") (unit 1) (value "1k8") (footprint "ukmarsbot:R_Axial_DIN0207_L6.3mm_D2.5mm_P7.62mm_Horizontal")
+      (reference "R5") (unit 1) (value "1k8") (footprint "ukmarsbot:R_Axial_DIN0207_L6.3mm_D2.5mm_P7.62mm_BIGPAD")
     )
     (path "/00000000-0000-0000-0000-000060ad9e54"
-      (reference "R6") (unit 1) (value "1k8") (footprint "ukmarsbot:R_Axial_DIN0207_L6.3mm_D2.5mm_P7.62mm_Horizontal")
+      (reference "R6") (unit 1) (value "1k8") (footprint "ukmarsbot:R_Axial_DIN0207_L6.3mm_D2.5mm_P7.62mm_BIGPAD")
     )
     (path "/00000000-0000-0000-0000-000060adb62e"
-      (reference "R7") (unit 1) (value "1k8") (footprint "ukmarsbot:R_Axial_DIN0207_L6.3mm_D2.5mm_P7.62mm_Horizontal")
+      (reference "R7") (unit 1) (value "1k8") (footprint "ukmarsbot:R_Axial_DIN0207_L6.3mm_D2.5mm_P7.62mm_BIGPAD")
     )
     (path "/00000000-0000-0000-0000-000060ad77e6"
-      (reference "R8") (unit 1) (value "1k8") (footprint "ukmarsbot:R_Axial_DIN0207_L6.3mm_D2.5mm_P7.62mm_Horizontal")
+      (reference "R8") (unit 1) (value "1k8") (footprint "ukmarsbot:R_Axial_DIN0207_L6.3mm_D2.5mm_P7.62mm_BIGPAD")
     )
     (path "/00000000-0000-0000-0000-000060ae73af"
-      (reference "R9") (unit 1) (value "100k") (footprint "ukmarsbot:R_Axial_DIN0207_L6.3mm_D2.5mm_P7.62mm_Horizontal")
+      (reference "R9") (unit 1) (value "100k") (footprint "ukmarsbot:R_Axial_DIN0207_L6.3mm_D2.5mm_P7.62mm_BIGPAD")
     )
     (path "/00000000-0000-0000-0000-000060af1d2d"
-      (reference "R10") (unit 1) (value "100k") (footprint "ukmarsbot:R_Axial_DIN0207_L6.3mm_D2.5mm_P7.62mm_Horizontal")
+      (reference "R10") (unit 1) (value "100k") (footprint "ukmarsbot:R_Axial_DIN0207_L6.3mm_D2.5mm_P7.62mm_BIGPAD")
     )
     (path "/00000000-0000-0000-0000-000060b75f9e"
-      (reference "R11") (unit 1) (value "33") (footprint "ukmarsbot:R_Axial_DIN0207_L6.3mm_D2.5mm_P7.62mm_Horizontal")
+      (reference "R11") (unit 1) (value "33") (footprint "ukmarsbot:R_Axial_DIN0207_L6.3mm_D2.5mm_P7.62mm_BIGPAD")
     )
     (path "/00000000-0000-0000-0000-000060b3feec"
-      (reference "R12") (unit 1) (value "1k0") (footprint "ukmarsbot:R_Axial_DIN0207_L6.3mm_D2.5mm_P7.62mm_Horizontal")
+      (reference "R12") (unit 1) (value "1k0") (footprint "ukmarsbot:R_Axial_DIN0207_L6.3mm_D2.5mm_P7.62mm_BIGPAD")
     )
     (path "/03379dcc-28e7-4b89-a687-1dd24e44f6e4"
-      (reference "R13") (unit 1) (value "390R") (footprint "ukmarsbot:R_Axial_DIN0207_L6.3mm_D2.5mm_P7.62mm_Horizontal")
+      (reference "R13") (unit 1) (value "390R") (footprint "ukmarsbot:R_Axial_DIN0207_L6.3mm_D2.5mm_P7.62mm_BIGPAD")
     )
     (path "/7edac8c3-b503-4b14-83f4-cb9aff87ff58"
-      (reference "R14") (unit 1) (value "390R") (footprint "ukmarsbot:R_Axial_DIN0207_L6.3mm_D2.5mm_P7.62mm_Horizontal")
-    )
-  )
+      (reference "R14") (unit 1) (value "390R") (footprint "ukmarsbot:R_Axial_DIN0207_L6.3mm_D2.5mm_P7.62mm_BIGPAD")
+    )
+  )

Commit message: update mounting holes on adv wall sensor
Parts:
- H1, H2: footprint MountingHole:MountingHole_2.7mm_Pad -> MountingHole:MountingHole_3.2mm_M3_Pad
Changed lines of the file:
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@@
       (effects (font (size 1.27 1.27)) (justify left))
     )
-    (property "Footprint" "MountingHole:MountingHole_2.7mm_Pad" (id 2) (at 41.91 43.18 0)
+    (property "Footprint" "MountingHole:MountingHole_3.2mm_M3_Pad" (id 2) (at 41.91 43.18 0)
       (effects (font (size 1.27 1.27)) hide)
     )
@@
       (effects (font (size 1.27 1.27)) (justify left))
     )
-    (property "Footprint" "MountingHole:MountingHole_2.7mm_Pad" (id 2) (at 41.91 55.88 0)
+    (property "Footprint" "MountingHole:MountingHole_3.2mm_M3_Pad" (id 2) (at 41.91 55.88 0)
       (effects (font (size 1.27 1.27)) hide)
     )
@@
     )
     (path "/00000000-0000-0000-0000-000060b03e53"
-      (reference "H1") (unit 1) (value "3.2mm") (footprint "MountingHole:MountingHole_2.7mm_Pad")
+      (reference "H1") (unit 1) (value "3.2mm") (footprint "MountingHole:MountingHole_3.2mm_M3_Pad")
     )
     (path "/00000000-0000-0000-0000-000060b04090"
-      (reference "H2") (unit 1) (value "3.2mm") (footprint "MountingHole:MountingHole_2.7mm_Pad")
+      (reference "H2") (unit 1) (value "3.2mm") (footprint "MountingHole:MountingHole_3.2mm_M3_Pad")
     )
     (path "/00000000-0000-0000-0000-000060b1cfe1"
