File: ecad/kicad/wall-sensor-advanced/ukmarsbot-wall-sensor-advanced.kicad_sch (KiCad schematic)
At the start: 30 parts, among them J1 Conn_01x14, Q1 TEFT4300, Q2 TEFT4300, Q3 TEFT4300, Q4 TEFT4300, Q5 BC337, Q6 BC337

Commit message: re-route and update adv wall sensor
Parts:
- D1, D2, D3, D4: Note (none) -> Ultra-bright red alternative but detectors must match
- D5: Note (none) -> Any small LED
- J1: Note (none) -> 14 way, 0.1" header chack polarity with mainboard
- Q1, Q2, Q3, Q4: Note (none) -> Spectral match to emitters
- Q5, Q6: Note (none) -> A MOSFET could be substitutes
- R1, R2, R3, R4: Note (none) -> Adjust on test according to emitters used
- R5, R6, R7, R8: Note (none) -> Adjust on test according to detectors used
Changed lines of the file:
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@@
+      (effects (font (size 1.27 1.27)) hide)
+    )
+    (property "Note" "Spectral match to emitters" (id 4) (at 189.23 50.8 0)
       (effects (font (size 1.27 1.27)) hide)
     )
@@
     )
     (property "Datasheet" "~" (id 3) (at 191.77 62.23 0)
+      (effects (font (size 1.27 1.27)) hide)
+    )
+    (property "Note" "Adjust on test according to detectors used" (id 4) (at 191.77 62.23 0)
       (effects (font (size 1.27 1.27)) hide)
     )
@@
       (effects (font (size 1.27 1.27)) hide)
     )
+    (property "Note" "Spectral match to emitters" (id 4) (at 146.05 50.8 0)
+      (effects (font (size 1.27 1.27)) hide)
+    )
     (pin "1")
     (pin "2")
@@
     )
     (property "Datasheet" "~" (id 3) (at 148.59 62.23 0)
+      (effects (font (size 1.27 1.27)) hide)
+    )
+    (property "Note" "Adjust on test according to detectors used" (id 4) (at 148.59 62.23 0)
       (effects (font (size 1.27 1.27)) hide)
     )
@@
       (effects (font (size 1.27 1.27)) hide)
     )
+    (property "Note" "Spectral match to emitters" (id 4) (at 167.64 50.8 0)
+      (effects (font (size 1.27 1.27)) hide)
+    )
     (pin "1")
     (pin "2")
@@
     )
     (property "Datasheet" "~" (id 3) (at 170.18 62.23 0)
+      (effects (font (size 1.27 1.27)) hide)
+    )
+    (property "Note" "Adjust on test according to detectors used" (id 4) (at 170.18 62.23 0)
       (effects (font (size 1.27 1.27)) hide)
     )
@@
       (effects (font (size 1.27 1.27)) hide)
     )
+    (property "Note" "Ultra-bright red alternative but detectors must match" (id 4) (at 184.15 121.92 0)
+      (effects (font (size 1.27 1.27)) hide)
+    )
     (pin "1")
     (pin "2")
@@
       (effects (font (size 1.27 1.27)) hide)
     )
+    (property "Note" "Adjust on test according to emitters used" (id 4) (at 184.15 111.76 0)
+      (effects (font (size 1.27 1.27)) hide)
+    )
     (pin "1")
     (pin "2")
@@
       (effects (font (size 1.27 1.27)) hide)
     )
+    (property "Note" "Ultra-bright red alternative but detectors must match" (id 4) (at 149.86 121.92 0)
+      (effects (font (size 1.27 1.27)) hide)
+    )
     (pin "1")
     (pin "2")
@@
     )
     (property "Datasheet" "~" (id 3) (at 149.86 111.76 0)
+      (effects (font (size 1.27 1.27)) hide)
+    )
+    (property "Note" "Adjust on test according to emitters used" (id 4) (at 149.86 111.76 0)
       (effects (font (size 1.27 1.27)) hide)
     )
@@
       (effects (font (size 1.27 1.27)) (justify left) hide)
     )
+    (property "Note" "A MOSFET could be substitutes" (id 4) (at 147.32 134.62 0)
+      (effects (font (size 1.27 1.27)) hide)
+    )
     (pin "1")
     (pin "2")
@@
       (effects (font (size 1.27 1.27)) hide)
     )
+    (property "Note" "Ultra-bright red alternative but detectors must match" (id 4) (at 135.89 121.92 0)
+      (effects (font (size 1.27 1.27)) hide)
+    )
     (pin "1")
     (pin "2")
@@
       (effects (font (size 1.27 1.27)) hide)
     )
+    (property "Note" "Adjust on test according to emitters used" (id 4) (at 135.89 111.76 0)
+      (effects (font (size 1.27 1.27)) hide)
+    )
     (pin "1")
     (pin "2")
@@
       (effects (font (size 1.27 1.27)) hide)
     )
+    (property "Note" "Ultra-bright red alternative but detectors must match" (id 4) (at 198.12 121.92 0)
+      (effects (font (size 1.27 1.27)) hide)
+    )
     (pin "1")
     (pin "2")
@@
       (effects (font (size 1.27 1.27)) hide)
     )
+    (property "Note" "Spectral match to emitters" (id 4) (at 124.46 50.8 0)
+      (effects (font (size 1.27 1.27)) hide)
+    )
     (pin "1")
     (pin "2")
@@
     )
     (property "Datasheet" "~" (id 3) (at 198.12 111.76 0)
+      (effects (font (size 1.27 1.27)) hide)
+    )
+    (property "Note" "Adjust on test according to emitters used" (id 4) (at 198.12 111.76 0)
       (effects (font (size 1.27 1.27)) hide)
     )
@@
       (effects (font (size 1.27 1.27)) (justify left) hide)
     )
+    (property "Note" "A MOSFET could be substitutes" (id 4) (at 195.58 134.62 0)
+      (effects (font (size 1.27 1.27)) hide)
+    )
     (pin "1")
     (pin "2")
@@
     )
     (property "Datasheet" "~" (id 3) (at 127 62.23 0)
+      (effects (font (size 1.27 1.27)) hide)
+    )
+    (property "Note" "Adjust on test according to detectors used" (id 4) (at 127 62.23 0)
       (effects (font (size 1.27 1.27)) hide)
     )
@@
     )
     (property "Datasheet" "~" (id 3) (at 26.67 100.33 0)
+      (effects (font (size 1.27 1.27)) hide)
+    )
+    (property "Note" "14 way, 0.1\" header chack polarity with mainboard" (id 4) (at 26.67 100.33 0)
       (effects (font (size 1.27 1.27)) hide)
     )
@@
       (effects (font (size 1.27 1.27)) hide)
     )
+    (property "Note" "Any small LED" (id 4) (at 41.91 162.56 0)
+      (effects (font (size 1.27 1.27)) hide)
+    )

Commit message: update emitter values in advanced wall sensor
Parts:
- D1, D2, D3, D4: value SFH4550 -> SFH4545
Other:
- note added: "Resistors R1, R2, R3 and R4 will be adjusted on test to suit the emitters in use. Current for the emitters is drawn from the capacitor C1. LEDs D1, D2, D3 and D4 may alternatively be high intensity red, blue or IR emitters. Whatever is chosen, take care that the detectors, Q3-6 are spectrally matched. An alternative to the SFH4545 IR emitters might be VSLY5940 or, for visible light, super bright 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"
- note removed: "Resistors R1, R2, R3 and R4 will be adjusted on test to suit the emitters in use. Current for the emitters is drawn from the capacitor C1. LEDs D1, D2, D3 and D4 may be high intensity red, blue or IR emitters. Whatever is chosen, take care that the detectors, Q3-6 are spectrally matched. An alternative to the SFH4550 IR emitters might be super bright red LEDs such as the TLCR5800 paired with BPW9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"
