File: ecad/kicad/line-sensor-mini-kes/line-sensor-mini-kes.kicad_sch (KiCad schematic)
At the start: 26 parts, among them J1 SENSORS, Q1 BC337, Q3 BPW85C, Q5 BPW85C, Q6 BPW85C, Q8 BPW85C

Commit message: update line-follower-mini-kes with KiCad project
Other:
- title: UKMARSBOT Line Sensor Mini -> UKMARSBOT Line Sensor Mini Kes
Changed lines of the file:
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@@
 	(paper "A4")
 	(title_block
-		(title "UKMARSBOT Line Sensor Mini")
+		(title "UKMARSBOT Line Sensor Mini Kes")
 		(date "2022-08-22")
 		(rev "1.0")
 		(company "UKMARS")
-		(comment 1 "Small line sensor for half size track")
+		(comment 1 "Small line sensor for Cytron Maker Nano ")
+		(comment 2 "David Hannaford")
 	)
 	(junction
